File: EAGLE/Technikerprojekt 2012/CNC-Controller.brd (EAGLE design)
At the start: 160 x 100 mm, 23 parts, among them IC1 mega1284P-PU, Q1 20MHz, X1 Einspeisung

Commit message: final SW version
Parts:
- removed U$1: MAX232_TI, max232ti:DIL16
- added AVRJTAG: JTAG, con-harting-ml:ML10
- added IC2: 7805TV, linear:TO220V
- added LED2: rot, led:LED3MM
- added R3: 330, resistor:0207/10
- added R4, R5: 10k, resistor:0207/10
- added U1: MAX232_TI, max232ti:DIL16
- AVRISP: value AVR-ISP-6 -> ISP; device avr-6:AVR-ISP-6 -> con-harting-ml:ML6
- B1: value 40V / 2A -> 35V / 4A; device rectifier:RB1A -> rectifier:KBU
- C1, C2: device rc-master:C025-050X025 -> rcl:C025-025X050
- Q1: value 20MHz -> 18.432MHz
- X1: value Einspeisung -> (none)
- moved RS232 134.0 mm to (14.0, 40.6), turned to 90 degrees
- moved C9 93.7 mm to (43.2, 69.8), turned to 90 degrees
- moved VDRIVE2 49.8 mm to (114.3, 17.8)
- moved GOCNC 33.5 mm to (114.3, 66.0)
- moved EDIP240-7 31.1 mm to (114.3, 40.6)
- moved C1 26.2 mm to (74.9, 50.8), turned to 180 degrees
- moved Q1 24.4 mm to (71.1, 44.5)
- moved C2 22.7 mm to (63.5, 50.8)
- moved C3 19.2 mm to (50.8, 69.8), turned to 270 degrees
- moved S1 18.5 mm to (67.3, 67.3), turned to 180 degrees
- moved X1 14.2 mm to (14.0, 72.4)
- moved R1 14.0 mm to (35.6, 64.8), turned to 0 degrees
- moved IC1 13.0 mm to (90.2, 50.8)
- moved LED1 11.7 mm to (34.3, 69.8), turned to 90 degrees
- moved C7 11.4 mm to (41.9, 33.0)
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Connections:
- net N$14 renamed UB-
- net N$9 renamed UB+
- removed net N$15: B1.-, C8.-
- removed net N$17: EDIP240-7.8
- removed net N$18: B1.+, C8.+
- removed net N$19: EDIP240-7.9
- new net PA7: GOCNC.8, IC1.33
- new net TCK: AVRJTAG.1, IC1.24
- new net TDI: AVRJTAG.9, IC1.27
- new net TDO: AVRJTAG.3, IC1.26
- new net TMS: AVRJTAG.5, IC1.25
- new net U+: B1.+, C8.+, IC2.1
- net GND: now also AVRJTAG.10, AVRJTAG.2, B1.-, C8.-, C9.-, EDIP240-7.7, EDIP240-7.8, GOCNC.10, IC2.2, R3.1, U1.15; no longer EDIP240-7.1, EDIP240-7.3, S1.4, U$1.15
- net N$10: now also U1.14; no longer U$1.14
- net N$11: now also U1.13; no longer U$1.13
- net N$12: now also U1.6; no longer U$1.6
- net N$13: now also IC1.19, LED2.A; no longer EDIP240-7.4
- net N$16: now also LED2.K, R3.2; no longer EDIP240-7.7
- net N$2: now also U1.1; no longer U$1.1
- net N$4: now also U1.3; no longer U$1.3
- net N$6: now also U1.4; no longer U$1.4
- net N$7: now also U1.5; no longer U$1.5
- net N$8: now also U1.2; no longer U$1.2
- net RST: now also AVRJTAG.6; no longer S1.2
- net RX0: now also U1.12; no longer U$1.12
- net SCL: now also R4.1
- net SDA: now also R5.1
- net TX0: now also U1.11; no longer U$1.11
- net VCC: now also AVRJTAG.4, AVRJTAG.7, C9.+, IC2.3, R4.2, R5.2, U1.16; no longer U$1.16
Routing:
- net GND: track 274.5 -> 19.4 mm, vias 0 -> 8
- net TDO: track 0.00 -> 94.0 mm
- net N$10: track 133.7 -> 47.6 mm
- net VCC: track 221.6 -> 303.5 mm
- net N$11: track 109.4 -> 44.0 mm
- net TCK: track 0.00 -> 61.3 mm
- net PA6: track 78.0 -> 16.8 mm
- net RX1: track 100.1 -> 40.9 mm
- net TDI: track 0.00 -> 58.2 mm
- net TMS: track 0.00 -> 56.2 mm, vias 0 -> 2
- net PA3: track 68.3 -> 18.3 mm
- net PA5: track 69.4 -> 19.4 mm
- net PA4: track 65.8 -> 15.8 mm
- net PA2: track 64.7 -> 15.8 mm
- net PA1: track 67.3 -> 19.4 mm
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- added copper zone on layer 1, net GND
- added copper zone on layer 16, net GND
Other:
- board size 160 x 100 mm -> 153.7 x 100 mm
- board text added: "12V"
- board text added: "AVRISP"
- board text added: "AVRJTAG"
- board text added: "CNC-Controller"
- board text added: "Dennis Hohmann"
- board text added: "RS232 DEBUG"
- board text added: "Reset"
- board text added: "Technikerarbeit 2012"
- board text added: "V1.0"
- board text added: "eDIP240-7"
- board text added: "goCNC"
- board text added: "vDRIVE2"
