File: EAGLE/Technikerprojekt 2012/CNC-Controller.sch (EAGLE design)
At the start: 23 parts, among them IC1 mega1284P-PU, Q1 20MHz, X1 Einspeisung

Commit message: final SW version
Parts:
- removed U$1: MAX232_TI, max232ti:MAX232_TI
- added AVRJTAG: JTAG, con-harting-ml:ML10
- added IC2: 7805TV, linear:7805TV
- added LED2: rot, led:LED3MM
- added R3: 330, resistor:R-EU_0207/10
- added R4, R5: 10k, resistor:R-EU_0207/10
- added U1: MAX232_TI, max232ti:MAX232_TI
- AVRISP: value AVR-ISP-6 -> ISP; device avr-6:AVR-ISP-6 -> con-harting-ml:ML6
- B1: value 40V / 2A -> 35V / 4A; device rectifier:RB1A -> rectifier:KBU
- C1, C2: device rc-master:C_C025-050X025 -> rcl:C-EU025-025X050
- Q1: value 20MHz -> 18.432MHz
- X1: value Einspeisung -> (none)
Connections:
- net N$14 renamed UB-
- net N$9 renamed UB+
- removed net N$15: B1.-, C8.-
- removed net N$17: EDIP240-7.8
- removed net N$18: B1.+, C8.+
- removed net N$19: EDIP240-7.9
- new net PA7: GOCNC.8, IC1.(ADC7/PCINT7)PA7
- new net TCK: AVRJTAG.1, IC1.(TCK/PCINT18)PC2
- new net TDI: AVRJTAG.9, IC1.(TDI/PCINT21)PC5
- new net TDO: AVRJTAG.3, IC1.(TDO/PCINT20)PC4
- new net TMS: AVRJTAG.5, IC1.(TMS/PCINT19)PC3
- new net U+: B1.+, C8.+, IC2.VI
- net GND: now also AVRJTAG.10, AVRJTAG.2, B1.-, C8.-, C9.-, EDIP240-7.7, EDIP240-7.8, GOCNC.10, IC2.GND, R3.1, U1.GND; no longer EDIP240-7.1, EDIP240-7.3, S1.P1, U$1.GND
- net N$10: now also U1.T1OUT; no longer U$1.T1OUT
- net N$11: now also U1.R1IN; no longer U$1.R1IN
- net N$12: now also U1.VS-; no longer U$1.VS-
- net N$13: now also IC1.(OC1A/PCINT29)PD5, LED2.A; no longer EDIP240-7.4
- net N$16: now also LED2.C, R3.2; no longer EDIP240-7.7
- net N$2: now also U1.C1+; no longer U$1.C1+
- net N$4: now also U1.C1-; no longer U$1.C1-
- net N$6: now also U1.C2+; no longer U$1.C2+
- net N$7: now also U1.C2-; no longer U$1.C2-
- net N$8: now also U1.VS+; no longer U$1.VS+
- net RST: now also AVRJTAG.6; no longer S1.S1
- net RX0: now also U1.R1OUT; no longer U$1.R1OUT
- net SCL: now also R4.1
- net SDA: now also R5.1
- net TX0: now also U1.T1IN; no longer U$1.T1IN
- net VCC: now also AVRJTAG.4, AVRJTAG.7, C9.+, IC2.VO, R4.2, R5.2, U1.VCC; no longer U$1.VCC
Other:
- note added: "1.00"
- note removed: "1.01"
- moved on the sheet: C1, C2, C3, C4, C5, C6, C7, C8, C9, IC1, LED1, Q1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
